File: tram_baseboard/tram_baseboard.kicad_pcb (KiCad board)
At the start: 4 copper layers, 160 x 100 mm, 23 parts, among them J1 Conn_01x04_Voltage, U1 SN74LVC2GU04, U6 SN74LVC1G06

Commit message: latest version 1 relaese with bugs
Parts:
- U2: footprint Connector_IDC:IDC-Header_2x05_P2.54mm_Vertical -> Connector_IDC:IDC-Header_2x05_P2.54mm_Horizontal
