File: tram_baseboard/tram_baseboard.kicad_pcb (KiCad board)
At the start: 4 copper layers, 160 x 100 mm, 23 parts, among them J1 Conn_01x04_Voltage, U1 SN74LVC2GU04, U6 SN74LVC1G06

Commit message: cleanup pluto
Parts:
- removed J1: Conn_01x04_Voltage, Transputer:PinHeader_1x04_P2.54mm_without_2
- added JP10: LinkOut, Connector_PinHeader_2.54mm:PinHeader_1x03_P2.54mm_Vertical, F.Cu at (66.7, 117.9)
- added JP3: SolderJumper_2_Bridged, Connector_PinHeader_2.54mm:PinHeader_1x02_P2.54mm_Vertical, F.Cu at (102.9, 94.5)
- added JP4: SolderJumper_2_Bridged, Connector_PinHeader_2.54mm:PinHeader_1x02_P2.54mm_Vertical, F.Cu at (102.9, 99.1)
- added JP5: SolderJumper_2_Bridged, Connector_PinHeader_2.54mm:PinHeader_1x02_P2.54mm_Vertical, F.Cu at (127.2, 74.9)
- added JP6: SolderJumper_2_Bridged, Connector_PinHeader_2.54mm:PinHeader_1x02_P2.54mm_Vertical, F.Cu at (131.8, 74.9)
- added JP7: SolderJumper_2_Bridged, Connector_PinHeader_2.54mm:PinHeader_1x02_P2.54mm_Vertical, F.Cu at (158.8, 39.9)
- added JP8: SolderJumper_2_Bridged, Connector_PinHeader_2.54mm:PinHeader_1x02_P2.54mm_Vertical, F.Cu at (158.8, 44.5)
- added JP9: Link_In, Connector_PinHeader_2.54mm:PinHeader_1x03_P2.54mm_Vertical, F.Cu at (71.2, 117.9)
- added R10: 10k, Resistor_SMD:R_0603_1608Metric_Pad0.98x0.95mm_HandSolder, F.Cu at (69.7, 42.5)
- added U4: SN74LVC1G04, Package_TO_SOT_SMD:SOT-23-5_HandSoldering, F.Cu at (65.4, 43.2)
- C1, R1: moved to B.Cu
- moved CON2 84.4 mm to (124.5, 34.3), turned to 180 degrees
- moved CON1 84.4 mm to (134.6, 118.1), turned to 0 degrees
- moved R8 9.89 mm to (191.0, 49.2)
- moved R1 9.35 mm to (199.1, 38.5), turned to 90 degrees
- moved JP1 7.80 mm to (196.8, 103.4)
- moved JP2 7.80 mm to (196.8, 108.0)
- moved C1 7.68 mm to (195.1, 38.3)
- moved LED1 7.03 mm to (56.8, 54.9)
- moved R4 7.03 mm to (66.2, 50.2)
- moved R5 7.03 mm to (63.7, 50.2)
- moved R6 4.08 mm to (191.0, 51.4)
- moved U6 3.36 mm to (60.0, 43.2)
- moved R7 3.36 mm to (191.0, 53.6)
- moved R9 2.05 mm to (191.0, 47.1)
Connections:
- CON0 pad 4: /Ext_LinkOut -> /LINK_T0_L1_OUT
- CON0 pad 5: /Ext_LinkIn -> /LINK_T0_L1_IN
- CON1 pad 4: Net-(CON0-LINK2IN) -> Net-(CON1-LINK1OUT)
- CON1 pad 5: Net-(CON0-LINK2OUT) -> Net-(CON1-LINK1IN)
- CON2 pad 4: Net-(CON1-LINK2IN) -> Net-(CON2-LINK1OUT)
- CON2 pad 5: Net-(CON1-LINK2OUT) -> Net-(CON2-LINK1IN)
- CON3 pad 4: Net-(CON2-LINK2IN) -> Net-(CON3-LINK1OUT)
- CON3 pad 5: Net-(CON2-LINK2OUT) -> Net-(CON3-LINK1IN)
- CON4 pad A10: /LINK_T2_L3_IN -> unconnected-(CON4-PadA10)
- CON4 pad A11: /LINK_T1_L3_OUT -> unconnected-(CON4-PadA11)
- CON4 pad A12: /LINK_T1_L3_IN -> unconnected-(CON4-PadA12)
- CON4 pad A13: /LINK_T0_L3_OUT -> unconnected-(CON4-PadA13)
- CON4 pad A14: /LINK_T0_L3_IN -> unconnected-(CON4-PadA14)
- CON4 pad A15: /LINK_T3_L2_OUT -> unconnected-(CON4-PadA15)
- CON4 pad A16: /LINK_T3_L2_IN -> unconnected-(CON4-PadA16)
- CON4 pad A2: +5V -> unconnected-(CON4-PadA2)
- CON4 pad A31: GND -> unconnected-(CON4-PadA31)
- CON4 pad A7: /LINK_T3_L3_OUT -> unconnected-(CON4-PadA7)
- CON4 pad A8: /LINK_T3_L3_IN -> unconnected-(CON4-PadA8)
- CON4 pad A9: /LINK_T2_L3_OUT -> unconnected-(CON4-PadA9)
- CON4 pad C10: /LINK_T2_L0_OUT -> unconnected-(CON4-PadC10)
- CON4 pad C11: /LINK_T1_L0_IN -> unconnected-(CON4-PadC11)
- CON4 pad C12: /LINK_T1_L0_OUT -> unconnected-(CON4-PadC12)
- CON4 pad C13: /LINK_T0_L0_IN -> unconnected-(CON4-PadC13)
- CON4 pad C14: /LINK_T0_L0_OUT -> unconnected-(CON4-PadC14)
- CON4 pad C2: +5V -> unconnected-(CON4-PadC2)
- CON4 pad C31: GND -> unconnected-(CON4-PadC31)
- CON4 pad C7: /LINK_T3_L0_IN -> unconnected-(CON4-PadC7)
- CON4 pad C8: /LINK_T3_L0_OUT -> unconnected-(CON4-PadC8)
- CON4 pad C9: /LINK_T2_L0_IN -> unconnected-(CON4-PadC9)
- U6 pad 2: /Ext_NotError -> Net-(U4-Pad4)
Routing:
- net /LinkSpeedB: track 254.8 -> 0.00 mm, vias 4 -> 0
- net /LinkSpeedA: track 249.5 -> 0.00 mm, vias 2 -> 0
- net /LINK_T0_L3_IN: track 163.2 -> 0.00 mm, vias 1 -> 0
- net /LINK_T0_L3_OUT: track 156.9 -> 0.00 mm, vias 1 -> 0
- net /LINK_T1_L0_OUT: track 138.1 -> 0.00 mm, vias 1 -> 0
- net /LINK_T1_L0_IN: track 137.1 -> 0.00 mm, vias 2 -> 0
- net /LINK_T1_L3_OUT: track 135.6 -> 0.00 mm, vias 1 -> 0
- net /LINK_T1_L3_IN: track 130.0 -> 0.00 mm, vias 1 -> 0
- net Net-(CON0-LINK2OUT): track 101.3 -> 0.00 mm
- net Net-(CON0-LINK2IN): track 100.2 -> 0.00 mm
- net /LINK_T2_L3_IN: track 98.9 -> 0.00 mm, vias 1 -> 0
- net /LINK_T2_L3_OUT: track 98.1 -> 0.00 mm, vias 1 -> 0
- net /LINK_T3_L0_OUT: track 94.8 -> 0.00 mm, vias 1 -> 0
- net Net-(CON1-LINK2IN): track 92.5 -> 0.00 mm
- net Net-(CON1-LINK2OUT): track 92.2 -> 0.00 mm
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Other:
- board text removed: "Nach Empfehlung Slot 0 2 1 3 -- Diskussion TJF 12.04.26"
