File: tram_baseboard/tram_baseboard.kicad_sch (KiCad schematic)
At the start: 23 parts, among them J1 Conn_01x04_Voltage, U1 SN74LVC2GU04, U6 SN74LVC1G06

Commit message: latest version 1 relaese with bugs
Parts:
- U2: footprint Connector_IDC:IDC-Header_2x05_P2.54mm_Vertical -> Connector_IDC:IDC-Header_2x05_P2.54mm_Horizontal
Other:
- title: (none) -> TRAM-Baseboard
Changed lines of the file:
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@@
 	(generator_version "9.0")
 	(paper "A4" portrait)
+	(title_block
+		(title "TRAM-Baseboard")
+		(date "2026-05-25")
+		(rev "1")
+	)
 	(bus_alias "Transputer_BUS"
 		(members "LinkSpeedA" "LinkSpeedB" "Clock_0" "Clock_1" "Clock_2" "Clock_3"
@@
 		)
 		(instances
-			(project "TRAM-Baseboard"
+			(project "tram_baseboard"
 				(path "/12343f12-7a98-419f-8ba8-29be77ce6edd"
 					(reference "R8")
@@
 		)
 		(instances
-			(project "TRAM-Baseboard"
+			(project "tram_baseboard"
 				(path "/12343f12-7a98-419f-8ba8-29be77ce6edd"
 					(reference "J1")
@@
 		)
 		(instances
-			(project "TRAM-Baseboard"
+			(project "tram_baseboard"
 				(path "/12343f12-7a98-419f-8ba8-29be77ce6edd"
 					(reference "#PWR065")
@@
 		)
 		(instances
-			(project "TRAM-Baseboard"
+			(project "tram_baseboard"
 				(path "/12343f12-7a98-419f-8ba8-29be77ce6edd"
 					(reference "#PWR04")
@@
 		)
 		(instances
-			(project "TRAM-Baseboard"
+			(project "tram_baseboard"
 				(path "/12343f12-7a98-419f-8ba8-29be77ce6edd"
 					(reference "#PWR07")
@@
 		)
 		(instances
-			(project "TRAM-Baseboard"
+			(project "tram_baseboard"
 				(path "/12343f12-7a98-419f-8ba8-29be77ce6edd"
 					(reference "R5")
@@
 		)
 		(instances
-			(project "TRAM-Baseboard"
+			(project "tram_baseboard"
 				(path "/12343f12-7a98-419f-8ba8-29be77ce6edd"
 					(reference "JP2")
@@
 		)
 		(instances
-			(project "TRAM-Baseboard"
+			(project "tram_baseboard"
 				(path "/12343f12-7a98-419f-8ba8-29be77ce6edd"
 					(reference "JP1")
@@
 		)
 		(instances
-			(project "TRAM-Baseboard"
+			(project "tram_baseboard"
 				(path "/12343f12-7a98-419f-8ba8-29be77ce6edd"
 					(reference "#PWR067")
@@
 		)
 		(instances
-			(project "TRAM-Baseboard"
+			(project "tram_baseboard"
 				(path "/12343f12-7a98-419f-8ba8-29be77ce6edd"
 					(reference "#PWR025")
@@
 		)
 		(instances
-			(project "TRAM-Baseboard"
+			(project "tram_baseboard"
 				(path "/12343f12-7a98-419f-8ba8-29be77ce6edd"
 					(reference "#PWR08")
@@
 		)
 		(instances
-			(project "TRAM-Baseboard"
+			(project "tram_baseboard"
 				(path "/12343f12-7a98-419f-8ba8-29be77ce6edd"
 					(reference "#FLG05")
@@
 		)
 		(instances
-			(project "TRAM-Baseboard"
+			(project "tram_baseboard"
 				(path "/12343f12-7a98-419f-8ba8-29be77ce6edd"
 					(reference "R9")
@@
 		)
 		(instances
-			(project "TRAM-Baseboard"
+			(project "tram_baseboard"
 				(path "/12343f12-7a98-419f-8ba8-29be77ce6edd"
 					(reference "CON2")
@@
 		)
 		(instances
-			(project "TRAM-Baseboard"
+			(project "tram_baseboard"
 				(path "/12343f12-7a98-419f-8ba8-29be77ce6edd"
 					(reference "R1")
@@
 		)
 		(instances
-			(project "TRAM-Baseboard"
+			(project "tram_baseboard"
 				(path "/12343f12-7a98-419f-8ba8-29be77ce6edd"
 					(reference "#PWR044")
@@
 		)
 		(instances
-			(project "TRAM-Baseboard"
+			(project "tram_baseboard"
 				(path "/12343f12-7a98-419f-8ba8-29be77ce6edd"
 					(reference "CON4")
@@
 		)
 		(instances
-			(project "TRAM-Baseboard"
+			(project "tram_baseboard"
 				(path "/12343f12-7a98-419f-8ba8-29be77ce6edd"
 					(reference "#PWR029")
@@
 		)
 		(instances
-			(project "TRAM-Baseboard"
+			(project "tram_baseboard"
 				(path "/12343f12-7a98-419f-8ba8-29be77ce6edd"
 					(reference "#PWR026")
@@
 		)
 		(instances
-			(project "TRAM-Baseboard"
+			(project "tram_baseboard"
 				(path "/12343f12-7a98-419f-8ba8-29be77ce6edd"
 					(reference "#PWR05")
@@
 		)
 		(instances
-			(project "TRAM-Baseboard"
+			(project "tram_baseboard"
 				(path "/12343f12-7a98-419f-8ba8-29be77ce6edd"
 					(reference "#FLG04")
@@
 		)
 		(instances
-			(project "TRAM-Baseboard"
+			(project "tram_baseboard"
 				(path "/12343f12-7a98-419f-8ba8-29be77ce6edd"
 					(reference "#PWR011")
@@
 		)
 		(instances
-			(project "TRAM-Baseboard"
+			(project "tram_baseboard"
 				(path "/12343f12-7a98-419f-8ba8-29be77ce6edd"
 					(reference "#PWR03")
@@
 		)
 		(instances
-			(project "TRAM-Baseboard"
+			(project "tram_baseboard"
 				(path "/12343f12-7a98-419f-8ba8-29be77ce6edd"
 					(reference "CON1")
@@
 		)
 		(instances
-			(project "TRAM-Baseboard"
+			(project "tram_baseboard"
 				(path "/12343f12-7a98-419f-8ba8-29be77ce6edd"
 					(reference "#PWR028")
@@
 		)
 		(instances
-			(project "TRAM-Baseboard"
+			(project "tram_baseboard"
 				(path "/12343f12-7a98-419f-8ba8-29be77ce6edd"
 					(reference "#PWR02")
@@
 		)
 		(instances
-			(project "TRAM-Baseboard"
+			(project "tram_baseboard"
 				(path "/12343f12-7a98-419f-8ba8-29be77ce6edd"
 					(reference "CON0")
@@
 		)
 		(instances
-			(project "TRAM-Baseboard"
+			(project "tram_baseboard"
 				(path "/12343f12-7a98-419f-8ba8-29be77ce6edd"
 					(reference "R6")
@@
 		)
 		(instances
-			(project "TRAM-Baseboard"
+			(project "tram_baseboard"
 				(path "/12343f12-7a98-419f-8ba8-29be77ce6edd"
 					(reference "C1")
@@
 		)
 		(instances
-			(project "TRAM-Baseboard"
+			(project "tram_baseboard"
 				(path "/12343f12-7a98-419f-8ba8-29be77ce6edd"
 					(reference "#PWR034")
@@
 		)
 		(instances
-			(project "TRAM-Baseboard"
+			(project "tram_baseboard"
 				(path "/12343f12-7a98-419f-8ba8-29be77ce6edd"
 					(reference "R7")
@@
 		)
 		(instances
-			(project "TRAM-Baseboard"
+			(project "tram_baseboard"
 				(path "/12343f12-7a98-419f-8ba8-29be77ce6edd"
 					(reference "#PWR066")
@@
 		)
 		(instances
-			(project "TRAM-Baseboard"
+			(project "tram_baseboard"
 				(path "/12343f12-7a98-419f-8ba8-29be77ce6edd"
 					(reference "CON3")
@@
 		)
 		(instances
-			(project "TRAM-Baseboard"
+			(project "tram_baseboard"
 				(path "/12343f12-7a98-419f-8ba8-29be77ce6edd"
 					(reference "#PWR09")
@@
 		)
 		(instances
-			(project "TRAM-Baseboard"
+			(project "tram_baseboard"
 				(path "/12343f12-7a98-419f-8ba8-29be77ce6edd"
 					(reference "#PWR06")
@@
 		)
 		(instances
-			(project "TRAM-Baseboard"
+			(project "tram_baseboard"
 				(path "/12343f12-7a98-419f-8ba8-29be77ce6edd"
 					(reference "#PWR023")
@@
 		)
 		(instances
-			(project "TRAM-Baseboard"
+			(project "tram_baseboard"
 				(path "/12343f12-7a98-419f-8ba8-29be77ce6edd"
 					(reference "QG2")
@@
 		)
 		(instances
-			(project "TRAM-Baseboard"
+			(project "tram_baseboard"
 				(path "/12343f12-7a98-419f-8ba8-29be77ce6edd"
 					(reference "#PWR048")
@@
 		)
 		(instances
-			(project "TRAM-Baseboard"
+			(project "tram_baseboard"
 				(path "/12343f12-7a98-419f-8ba8-29be77ce6edd"
 					(reference "#PWR033")
@@
 		)
 		(instances
-			(project "TRAM-Baseboard"
+			(project "tram_baseboard"
 				(path "/12343f12-7a98-419f-8ba8-29be77ce6edd"
 					(reference "LED1")
@@
 		)
 		(instances
-			(project "TRAM-Baseboard"
+			(project "tram_baseboard"
 				(path "/12343f12-7a98-419f-8ba8-29be77ce6edd"
 					(reference "#PWR040")
@@
 		)
 		(instances
-			(project "TRAM-Baseboard"
+			(project "tram_baseboard"
 				(path "/12343f12-7a98-419f-8ba8-29be77ce6edd"
 					(reference "U6")
@@
 			)
 		)
-		(property "Footprint" "Connector_IDC:IDC-Header_2x05_P2.54mm_Vertical"
+		(property "Footprint" "Connector_IDC:IDC-Header_2x05_P2.54mm_Horizontal"
 			(at 15.494 191.008 90)
 			(effects
@@
 		)
 		(instances
-			(project "TRAM-Baseboard"
+			(project "tram_baseboard"
 				(path "/12343f12-7a98-419f-8ba8-29be77ce6edd"
 					(reference "U2")
@@
 		)
 		(instances
-			(project "TRAM-Baseboard"
+			(project "tram_baseboard"
 				(path "/12343f12-7a98-419f-8ba8-29be77ce6edd"
 					(reference "#PWR070")
@@
 		)
 		(instances
-			(project "TRAM-Baseboard"
+			(project "tram_baseboard"
 				(path "/12343f12-7a98-419f-8ba8-29be77ce6edd"
 					(reference "#PWR068")
@@
 		)
 		(instances
-			(project "TRAM-Baseboard"
+			(project "tram_baseboard"
 				(path "/12343f12-7a98-419f-8ba8-29be77ce6edd"
 					(reference "#PWR018")
@@
 		)
 		(instances
-			(project "TRAM-Baseboard"
+			(project "tram_baseboard"
 				(path "/12343f12-7a98-419f-8ba8-29be77ce6edd"
 					(reference "R4")
@@
 		)
 		(instances
-			(project "TRAM-Baseboard"
+			(project "tram_baseboard"
 				(path "/12343f12-7a98-419f-8ba8-29be77ce6edd"
 					(reference "U1")
@@
 		)
 		(instances
-			(project "TRAM-Baseboard"
+			(project "tram_baseboard"
 				(path "/12343f12-7a98-419f-8ba8-29be77ce6edd"
 					(reference "#PWR01")
@@
 		)
 		(instances
-			(project "TRAM-Baseboard"
+			(project "tram_baseboard"
 				(path "/12343f12-7a98-419f-8ba8-29be77ce6edd"
 					(reference "#PWR027")
@@
 		)
 		(instances
-			(project "TRAM-Baseboard"
+			(project "tram_baseboard"
 				(path "/12343f12-7a98-419f-8ba8-29be77ce6edd"
 					(reference "#PWR043")
@@
 		)
 		(instances
-			(project "TRAM-Baseboard"
+			(project "tram_baseboard"
 				(path "/12343f12-7a98-419f-8ba8-29be77ce6edd"
 					(reference "#PWR069")
@@
 		)
 		(instances
-			(project "TRAM-Baseboard"
+			(project "tram_baseboard"
 				(path "/12343f12-7a98-419f-8ba8-29be77ce6edd"
 					(reference "#PWR030")
@@
 		)
 		(instances
-			(project "TRAM-Baseboard"
+			(project "tram_baseboard"
 				(path "/12343f12-7a98-419f-8ba8-29be77ce6edd"
 					(reference "R3")
@@
 		)
 		(instances
-			(project "TRAM-Baseboard"
+			(project "tram_baseboard"
 				(path "/12343f12-7a98-419f-8ba8-29be77ce6edd"
 					(reference "R2")
@@
 		)
 		(instances
-			(project "TRAM-Baseboard"
+			(project "tram_baseboard"
 				(path "/12343f12-7a98-419f-8ba8-29be77ce6edd"
 					(reference "#PWR024")
