File: tram_baseboard/tram_baseboard.kicad_sch (KiCad schematic)
At the start: 23 parts, among them J1 Conn_01x04_Voltage, U1 SN74LVC2GU04, U6 SN74LVC1G06

Commit message: cleanup pluto
Parts:
- removed J1: Conn_01x04_Voltage, Transputer:PinHeader_1x04_P2.54mm_without_2, symbol Transputer:Conn_01x04_Voltage
- added JP10: LinkOut, Connector_PinHeader_2.54mm:PinHeader_1x03_P2.54mm_Vertical, symbol Jumper:Jumper_3_Open
- added JP3, JP4, JP5, JP6, JP7, JP8: SolderJumper_2_Bridged, Connector_PinHeader_2.54mm:PinHeader_1x02_P2.54mm_Vertical, symbol Jumper:SolderJumper_2_Bridged
- added JP9: Link_In, Connector_PinHeader_2.54mm:PinHeader_1x03_P2.54mm_Vertical, symbol Jumper:Jumper_3_Open
- added R10: 10k, Resistor_SMD:R_0603_1608Metric_Pad0.98x0.95mm_HandSolder, symbol Device:R_Small
- added U4: SN74LVC1G04, Package_TO_SOT_SMD:SOT-23-5_HandSoldering, symbol Transputer:SN74LVC1G04
- CON0, CON1, CON2, CON3, CON4, LED1, QG2, U2: value ~ -> (none)
Connections:
- net +5V: now also R10.1, U4.5 (VCC); no longer CON4.A2, CON4.C2
- net Ext_LinkIn: now also JP9.2 (C); no longer CON0.5 (LINK1IN)
- net Ext_LinkOut: now also JP10.2 (C); no longer CON0.4 (LINK1OUT)
- net Ext_NotError: now also R10.2, U4.2; no longer U6.2
- net GND: now also U4.3 (GND); no longer CON4.A31, CON4.C31
- net LINK_T0_L0_IN: now also JP9.3 (B); no longer CON4.C13
- net LINK_T0_L0_OUT: now also JP10.3 (B); no longer CON4.C14
- net LINK_T0_L3_IN: no longer CON4.A14
- net LINK_T0_L3_OUT: no longer CON4.A13
- net LINK_T1_L0_IN: no longer CON4.C11
- net LINK_T1_L0_OUT: no longer CON4.C12
- net LINK_T1_L3_IN: no longer CON4.A12
- net LINK_T1_L3_OUT: no longer CON4.A11
- net LINK_T2_L0_IN: no longer CON4.C9
- net LINK_T2_L0_OUT: no longer CON4.C10
- net LINK_T2_L3_IN: no longer CON4.A10
- net LINK_T2_L3_OUT: no longer CON4.A9
- net LINK_T3_L0_IN: no longer CON4.C7
- net LINK_T3_L0_OUT: no longer CON4.C8
- net LINK_T3_L2_IN: no longer CON4.A16
- net LINK_T3_L2_OUT: no longer CON4.A15
- net LINK_T3_L3_IN: no longer CON4.A8
- net LINK_T3_L3_OUT: no longer CON4.A7
- net at CON2.1 (LINK2OUT): now also JP7.2 (B); no longer CON3.5 (LINK1IN)
- net at CON3.4 (LINK1OUT): now also JP8.1 (A); no longer CON2.2 (LINK2IN)
- net at CON2.4 (LINK1OUT): now also JP6.1 (A); no longer CON1.2 (LINK2IN)
- net at CON2.5 (LINK1IN): now also JP5.1 (A); no longer CON1.1 (LINK2OUT)
- net at CON1.4 (LINK1OUT): now also JP4.1 (A); no longer CON0.2 (LINK2IN)
- net at CON1.5 (LINK1IN): now also JP3.1 (A); no longer CON0.1 (LINK2OUT)
- new net: CON2.2 (LINK2IN), JP8.2 (B)
- new net: CON1.1 (LINK2OUT), JP5.2 (B)
- new net: CON1.2 (LINK2IN), JP6.2 (B)
- new net: CON0.1 (LINK2OUT), JP3.2 (B)
- new net: CON0.2 (LINK2IN), JP4.2 (B)
- new net: U4.4, U6.2
- new net: CON3.5 (LINK1IN), JP7.1 (A)
- new net LINK_T0_L1_IN: CON0.5 (LINK1IN), JP9.1 (A)
- new net LINK_T0_L1_OUT: CON0.4 (LINK1OUT), JP10.1 (A)
- no-connect marks 40 -> 39
Other:
- note removed: "Hier ist auf jeden Fall ein Fehler, G04 muss davor, dann passt die Logic und 10 k nach 5 V"
- company: (none) -> dg1vs-labs
- moved on the sheet: C1, CON0, CON1, CON2, CON3, CON4, JP1, JP2, LED1, QG2, R1, R2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
